File: breakouts/W3113/W3113.brd (EAGLE design)
At the start: 14 x 13.5 mm, 3 parts

Commit message: W3113 adjustments
Parts:
- moved E$1 1.00 mm to (9.00, 3.00)
- moved E$2 1.00 mm to (7.00, 3.00)
- moved E$3 1.00 mm to (16.0, 3.00)
Routing:
- net S$2: track 4.21 -> 5.41 mm
Other:
- board size 14 x 13.5 mm -> 15 x 17 mm
Changed lines of the file:
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@@
 <?xml version="1.0" encoding="utf-8"?>
 <!DOCTYPE eagle SYSTEM "eagle.dtd">
-<eagle version="6.2">
+<eagle version="6.3">
 <drawing>
 <settings>
@@
 <board>
 <plain>
-<rectangle x1="5" y1="6.5" x2="18" y2="14.5" layer="39"/>
+<rectangle x1="5" y1="6.5" x2="18" y2="16.5" layer="39"/>
 <rectangle x1="5.5" y1="6.5" x2="8.5" y2="8" layer="1"/>
-<wire x1="4.5" y1="1.5" x2="18.5" y2="1.5" width="0.4064" layer="20"/>
-<wire x1="18.5" y1="1.5" x2="18.5" y2="15" width="0.4064" layer="20"/>
-<wire x1="18.5" y1="15" x2="4.5" y2="15" width="0.4064" layer="20"/>
-<wire x1="4.5" y1="15" x2="4.5" y2="1.5" width="0.4064" layer="20"/>
+<wire x1="4" y1="0.5" x2="19" y2="0.5" width="0.4064" layer="20"/>
+<wire x1="19" y1="0.5" x2="19" y2="17.5" width="0.4064" layer="20"/>
+<wire x1="19" y1="17.5" x2="4" y2="17.5" width="0.4064" layer="20"/>
+<wire x1="4" y1="17.5" x2="4" y2="0.5" width="0.4064" layer="20"/>
 <text x="17" y="10.5" size="1.4224" layer="122" font="vector" rot="MR0">quilix.com</text>
-<rectangle x1="5" y1="6.5" x2="18" y2="14.5" layer="41"/>
+<rectangle x1="5" y1="6.5" x2="18" y2="16.5" layer="41"/>
 </plain>
 <attributes>
@@
 </class>
 </classes>
-<designrules>
+<designrules name="default">
 <description language="de">&lt;b&gt;EAGLE Design Rules&lt;/b&gt;
 &lt;p&gt;
@@
 </autorouter>
 <elements>
-<element name="E$1" library="SparkFun" package="SMA-EDGE" value="" x="9" y="4"/>
-<element name="E$2" library="adafruit" package="1X01-CLEANBIG" value="" x="7" y="4"/>
-<element name="E$3" library="adafruit" package="1X01-CLEANBIG" value="" x="16" y="4"/>
+<element name="E$1" library="SparkFun" package="SMA-EDGE" value="" x="9" y="3"/>
+<element name="E$2" library="adafruit" package="1X01-CLEANBIG" value="" x="7" y="3"/>
+<element name="E$3" library="adafruit" package="1X01-CLEANBIG" value="" x="16" y="3"/>
 </elements>
 <signals>
 <signal name="S$2">
-<wire x1="11.5" y1="5.5" x2="11.5" y2="6.5" width="0.4064" layer="1"/>
-<wire x1="11.5" y1="6.5" x2="11" y2="7" width="0.4064" layer="1"/>
-<wire x1="11" y1="7" x2="8.5" y2="7" width="0.4064" layer="1"/>
+<wire x1="11.5" y1="4.5" x2="11.5" y2="6" width="0.4064" layer="1"/>
+<wire x1="11.5" y1="6" x2="9" y2="6" width="0.4064" layer="1"/>
+<wire x1="9" y1="6" x2="8" y2="7" width="0.4064" layer="1"/>
 </signal>
 <signal name="ANT">
-<wire x1="7.5" y1="4" x2="9" y2="4" width="0.6096" layer="1"/>
-<wire x1="14" y1="4" x2="15.5" y2="4" width="0.6096" layer="1"/>
-<wire x1="9" y1="4" x2="14" y2="4" width="0" layer="19" extent="1-1"/>
-<wire x1="7.5" y1="4" x2="9" y2="4" width="0.6096" layer="16"/>
-<wire x1="14" y1="4" x2="15.5" y2="4" width="0.6096" layer="16"/>
+<wire x1="7.5" y1="3" x2="9" y2="3" width="0.6096" layer="1"/>
+<wire x1="14" y1="3" x2="15.5" y2="3" width="0.6096" layer="1"/>
+<wire x1="9" y1="3" x2="14" y2="3" width="0" layer="19" extent="1-1"/>
+<wire x1="7.5" y1="3" x2="9" y2="3" width="0.6096" layer="16"/>
+<wire x1="14" y1="3" x2="15.5" y2="3" width="0.6096" layer="16"/>
 </signal>
 </signals>
