File: breakouts/CRYSTALATOR/CRYSTALATOR.brd (EAGLE design)
At the start: 18 x 21 mm, 10 parts

Commit message: The New CRYSTALATOR!
Now with bigger capacitor footprints! 1206 to be exact.
Parts:
- E$5, E$6: device adafruit:C0805K -> adafruit:C1206
Changed lines of the file:
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@@
 <element name="E$4" library="SparkFun" package="CAP-PTH-SMALL" value="" x="22" y="7.3" rot="R90"/>
 <element name="E$1" library="SparkFun" package="HC49U-V" value="" x="17.05" y="14.6"/>
-<element name="E$5" library="adafruit" package="C0805K" value="" x="9.7" y="8.5" rot="R90"/>
-<element name="E$6" library="adafruit" package="C0805K" value="" x="24.35" y="8.55" rot="R90"/>
+<element name="E$5" library="adafruit" package="C1206" value="" x="9.7" y="8.5" rot="R90"/>
+<element name="E$6" library="adafruit" package="C1206" value="" x="24.35" y="8.55" rot="R90"/>
 </elements>
 <signals>
@@
 <wire x1="14.65" y1="17.713" x2="14.65" y2="21.65" width="0.3048" layer="1"/>
 <wire x1="12" y1="7.25" x2="9.7" y2="7.25" width="0.3048" layer="1"/>
-<wire x1="9.7" y1="7.25" x2="9.7" y2="7.5" width="0.3048" layer="1"/>
+<wire x1="9.7" y1="7.25" x2="9.7" y2="7.1" width="0.3048" layer="1"/>
 <wire x1="12" y1="7.25" x2="15.2" y2="7.25" width="0.3048" layer="1"/>
 <wire x1="15.2" y1="7.25" x2="15.2" y2="7.45" width="0.3048" layer="1"/>
@@
 <wire x1="18.99" y1="9.84" x2="22" y2="9.84" width="0.3048" layer="1"/>
 <wire x1="22" y1="9.84" x2="24.35" y2="9.84" width="0.3048" layer="1"/>
-<wire x1="24.35" y1="9.84" x2="24.35" y2="9.55" width="0.3048" layer="1"/>
+<wire x1="24.35" y1="9.84" x2="24.35" y2="9.95" width="0.3048" layer="1"/>
 <wire x1="19.463" y1="14.6" x2="19.55" y2="14.487" width="0.3048" layer="1"/>
 <wire x1="19.55" y1="14.487" x2="19.55" y2="9.75" width="0.3048" layer="1"/>
@@
 <contactref element="E$6" pad="1"/>
 <wire x1="22" y1="7.3" x2="24.35" y2="7.3" width="0.3048" layer="1"/>
-<wire x1="24.35" y1="7.3" x2="24.35" y2="7.55" width="0.3048" layer="1"/>
+<wire x1="24.35" y1="7.3" x2="24.35" y2="7.15" width="0.3048" layer="1"/>
 <wire x1="12" y1="9.79" x2="9.7" y2="9.79" width="0.3048" layer="1"/>
-<wire x1="9.7" y1="9.79" x2="9.7" y2="9.5" width="0.3048" layer="1"/>
+<wire x1="9.7" y1="9.79" x2="9.7" y2="9.9" width="0.3048" layer="1"/>
 <wire x1="12" y1="9.79" x2="17.06991875" y2="8.527590625" width="0.3048" layer="16"/>
 <wire x1="17.06991875" y1="8.527590625" x2="22" y2="7.3" width="0.3048" layer="16"/>
