File: Adapters/ISP2DIP/ISP2DIP.brd (EAGLE design)
At the start: 39 x 12.9 mm, 4 parts

Commit message: cam, loop, and gerbers update
Parts:
- moved E$1 20.5 mm to (37.2, 9.98)
- moved E$2 20.5 mm to (22.5, 9.98)
- moved E$4 20.5 mm to (7.99, 13.8)
- moved E$5 20.5 mm to (7.99, 6.17)
Other:
- board size 39 x 12.9 mm -> 41.5 x 12.9 mm
